File: DS8641N_tester.kicad_pcb (KiCad board)
At the start: 2 copper layers, 76.2 x 65.4 mm, 39 parts, among them J1 Barrel_Jack, J2 Conn_01x05_Pin, J4 Conn_01x05_Pin, SW1 Bus 1, SW2 Bus 2, SW3 Bus 3, SW4 Bus 4, SW5 DISABLE A, SW6 DISABLE B, U1 DS8641N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

Commit message: Added image and small fix
Parts:
- removed R6, R7: 10k, Resistor_THT:R_Axial_DIN0204_L3.6mm_D1.6mm_P7.62mm_Horizontal
- SW5: value DISABLE A -> ENABLE A
- SW6: value DISABLE B -> ENABLE B
Connections:
- SW5 pad 1: +5V -> GND
- SW6 pad 1: +5V -> GND
Routing:
- net Net-(SW6-Pad2): track 36.1 -> 27.8 mm
- net Net-(SW5-Pad2): track 45.2 -> 43.0 mm
- net +5V: track 176.5 -> 178.0 mm
Other:
- board text added: "&"
- board text added: "Rev B"
- board text removed: "Rev A"
