File: DS8641N_tester.kicad_sch (KiCad schematic)
At the start: 39 parts, among them J1 Barrel_Jack, J2 Conn_01x05_Pin, J4 Conn_01x05_Pin, SW1 Bus 1, SW2 Bus 2, SW3 Bus 3, SW4 Bus 4, SW5 DISABLE A, SW6 DISABLE B, U1 DS8641N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

Commit message: Added image and small fix
Parts:
- removed R6, R7: 10k, Resistor_THT:R_Axial_DIN0204_L3.6mm_D1.6mm_P7.62mm_Horizontal, symbol Device:R
Connections:
- net +5V: no longer SW5.1, SW6.1
- net GND: now also SW5.1, SW6.1
